File: hellen64_NA8_96.kicad_sch (KiCad schematic)
At the start: 192 parts, among them J1 USB_B_Mini, J11 Conn_01x01, J13 Conn_01x01, J14 Conn_01x01, J15 Conn_01x01, J16 Conn_01x01, J17 Conn_01x01, J19 Conn_01x01, J2 Conn_01x05_Male, J20 Conn_01x01, J21 Conn_01x01, J22 Conn_01x01, J24 Conn_01x01, J25 AudioJack3_SwitchTR, J27 Conn_01x06, J3 MiniFit, J4 Conn_02x12_Odd_Even, J5 USB_B, J6 ETB, M1 Module-input-0.1, M10 Module-power12-0.2, M11 Module-power5-0.2, M12 Module-wbo-0.2, M13 Module-can-0.1, M2 Module-ign8-0.1, M3 Module-mcu144-0.5, M4 Module-sd-0.1, M5 Module-output-0.2, M6 Module-dinput4-0.1, M7 Module-stlink-0.1, M8 Module-can-0.1, M9 Module-knock-0.1, P1 Pad, P10 Pad, P11 Pad, P12 Pad, P13 Pad, P14 Pad, P15 Pad, P17 Pad, P18 Pad, P19 Pad, P2 178780-1, P20 Pad, P22 Pad, P23 Pad, P24 Pad, P25 Pad, P28 Pad, P29 Pad, P30 Pad, P31 Pad, P32 Pad, P38 Pad, P4 Pad, P43 Pad, P44 Pad, P47 Pad, P48 Pad, P49 Pad, P5 Pad, P50 Pad, P51 Pad, P52 Pad, P53 Pad, P55 Pad, P56 Pad, P6 Pad, P7 Pad, P8 Pad, P9 Pad, U1 LIS2DW12TR, U2 MPX4_MAP, U3 MCP6002-xSN, U4 LPS25HB, U5 L6205PD

Commit message: update schematics
Parts:
- removed R20, R22, R28, R30, R33, R34, R36, R47, R49, R8: Jumper-Pad-Pad, hellen-one-common:PAD-0805-PAD, symbol hellen-one-common:Jumper-Pad-Pad
- added P16, P21, P26, P27, P3, P33: Pad, hellen-one-common:PAD-TH, symbol hellen-one-common:Pad
Connections:
- net IN_VIGN is gone; now on net +12V_RAW: D10.1 (A), D5.1 (K), M10.V3 (IN_VIGN)
- net 1B: no longer F2.2
- net 1Q: no longer M5.S13 (OUT_LOW12)
- net 1V: now also P16.1 (Pin_1)
- net 3B: now also F2.2
- net 3J: now also P3.1 (Pin_1)
- net 3S: now also R27.1; no longer P53.1 (Pin_1)
- net IN_EGR_BOOST: now also R27.2
- net IN_IAT: no longer M5.S6 (OUT_PP2), R24.1
- net IN_KNOCK_RAW: now also P2.10 (1S); no longer J6.2 (Pin_2), M1.S10 (IN_TPS), P2.33 (2F)
- net IN_MAP: now also P26.1 (Pin_1)
- net IN_NEUTRAL: now also P33.1 (Pin_1)
- net IN_PRESSURE: now also R18.1
- net IN_STEERING: now also P27.1 (Pin_1)
- net OUT_IDLE: no longer D31.2 (A), M5.W11 (OUT_INJ8)
- net OUT_IGN1: no longer D17.2 (K), D21.2 (A), M5.S14 (OUT_LOW9), M5.S7 (OUT_LOW3_DUAL), R26.1, R32.1
- net OUT_INJ2: no longer M5.W4 (OUT_LOW4_DUAL), R25.1
- net at P2.23 (2A): now also R18.2
- net 4C: now reaches P2.66 (4C), R21.2
- net 4D: now reaches P2.72 (4D), R43.2
- net at P2.20 (1R): now also P21.1 (Pin_1)
- net at P2.59 (3P): now also P53.1 (Pin_1)
- new net IN_TPS: J6.2 (Pin_2), M1.S10 (IN_TPS), P2.33 (2F)
- new net OUT_O2H: M5.S7 (OUT_LOW3_DUAL), R26.1
- new net OUT_O2H2: M5.W4 (OUT_LOW4_DUAL), R25.1
- new net OUT_PUMP_RELAY: D17.2 (K), D21.2 (A), M5.S14 (OUT_LOW9), R32.1
- new net OUT_TACH: M5.S6 (OUT_PP2), R24.1
- new net OUT_VICS: D31.2 (A), M5.W11 (OUT_INJ8)
Other:
- note removed: "Currently unused:"
- moved on the sheet: P47, P48, P49, P50, P51, P53, P56, P7, R18, R27

Commit message: pcb progress
Parts:
- added P34, P35, P36: Pad, hellen-one-common:PAD-TH, symbol hellen-one-common:Pad
- added R8: Jumper-Pad-Pad, hellen-one-common:PAD-0805-PAD, symbol hellen-one-common:Jumper-Pad-Pad
Connections:
- net 3R: now also R8.2; no longer D4.1 (A), M2.S7 (OUT_IGN2)
- net IN_O2S3: now also P36.1 (Pin_1)
- net at M5.S13 (OUT_LOW12): now also P34.1 (Pin_1)
- net OUT_ALTERNATOR renamed OUT_PP1
- net OUT_PP1: now also P35.1 (Pin_1)
- new net OUT_IGN2: D4.1 (A), M2.S7 (OUT_IGN2), R8.1
Changed lines of the file:
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@@
     (stroke (width 0.1524) (type solid) (color 0 0 0 0))
   )
-  (bus_entry (at 275.59 280.67) (size -2.54 2.54)
-    (stroke (width 0.1524) (type solid) (color 0 0 0 0))
-  )
   (bus_entry (at 284.48 71.12) (size -2.54 2.54)
     (stroke (width 0.1524) (type solid) (color 0 0 0 0))
@@
     (stroke (width 0) (type solid) (color 0 0 0 0))
   )
-  (wire (pts (xy 93.98 95.25) (xy 210.82 95.25))
+  (wire (pts (xy 93.98 95.25) (xy 105.41 95.25))
     (stroke (width 0) (type solid) (color 0 0 0 0))
   )
@@
     (stroke (width 0) (type solid) (color 0 0 0 0))
   )
+  (wire (pts (xy 115.57 95.25) (xy 210.82 95.25))
+    (stroke (width 0) (type solid) (color 0 0 0 0))
+  )
   (wire (pts (xy 115.57 105.41) (xy 210.82 105.41))
     (stroke (width 0) (type solid) (color 0 0 0 0))
@@
     (stroke (width 0) (type solid) (color 0 0 0 0))
   )
-  (wire (pts (xy 234.95 168.91) (xy 309.88 168.91))
-    (stroke (width 0) (type solid) (color 0 0 0 0))
-  )
   (wire (pts (xy 236.22 106.68) (xy 236.22 113.03))
     (stroke (width 0) (type solid) (color 0 0 0 0))
@@
     (stroke (width 0) (type solid) (color 0 0 0 0))
   )
-  (wire (pts (xy 264.16 139.7) (xy 264.16 158.75))
-    (stroke (width 0) (type solid) (color 0 0 0 0))
-  )
   (wire (pts (xy 264.16 139.7) (xy 309.88 139.7))
     (stroke (width 0) (type solid) (color 0 0 0 0))
   )
-  (wire (pts (xy 266.7 116.84) (xy 266.7 166.37))
-    (stroke (width 0) (type solid) (color 0 0 0 0))
-  )
-  (wire (pts (xy 266.7 116.84) (xy 309.88 116.84))
-    (stroke (width 0) (type solid) (color 0 0 0 0))
-  )
   (wire (pts (xy 266.7 353.06) (xy 267.97 353.06))
     (stroke (width 0) (type solid) (color 0 0 0 0))
@@
     (stroke (width 0) (type solid) (color 0 0 0 0))
   )
-  (wire (pts (xy 269.24 142.24) (xy 269.24 181.61))
-    (stroke (width 0) (type solid) (color 0 0 0 0))
-  )
   (wire (pts (xy 269.24 142.24) (xy 309.88 142.24))
     (stroke (width 0) (type solid) (color 0 0 0 0))
@@
     (stroke (width 0) (type solid) (color 0 0 0 0))
   )
-  (wire (pts (xy 275.59 280.67) (xy 309.88 280.67))
-    (stroke (width 0) (type solid) (color 0 0 0 0))
-  )
   (wire (pts (xy 275.59 321.31) (xy 293.37 321.31))
     (stroke (width 0) (type solid) (color 0 0 0 0))
@@
     (stroke (width 0) (type solid) (color 0 0 0 0))
   )
+  (wire (pts (xy 290.83 116.84) (xy 309.88 116.84))
+    (stroke (width 0) (type solid) (color 0 0 0 0))
+  )
+  (wire (pts (xy 290.83 167.64) (xy 309.88 167.64))
+    (stroke (width 0) (type solid) (color 0 0 0 0))
+  )
   (wire (pts (xy 290.83 172.72) (xy 309.88 172.72))
     (stroke (width 0) (type solid) (color 0 0 0 0))
@@
     (stroke (width 0) (type solid) (color 0 0 0 0))
   )
+  (wire (pts (xy 294.64 280.67) (xy 309.88 280.67))
+    (stroke (width 0) (type solid) (color 0 0 0 0))
+  )
   (wire (pts (xy 295.91 300.99) (xy 309.88 300.99))
     (stroke (width 0) (type solid) (color 0 0 0 0))
@@
     (stroke (width 0) (type solid) (color 0 0 0 0))
   )
-  (wire (pts (xy 309.88 168.91) (xy 309.88 167.64))
-    (stroke (width 0) (type solid) (color 0 0 0 0))
-  )
   (wire (pts (xy 309.88 195.58) (xy 309.88 198.12))
     (stroke (width 0) (type solid) (color 0 0 0 0))
@@
     (effects (font (size 1.27 1.27)) (justify right bottom))
   )
-  (label "OUT_ALTERNATOR" (at 307.34 116.84 180)
+  (label "OUT_PP1" (at 307.34 116.84 180)
     (effects (font (size 1.27 1.27)) (justify right bottom))
   )
@@
     (pin "1")
   )
+  (symbol (lib_id "hellen-one-common:Pad") (at 285.75 116.84 0) (mirror y) (unit 1)
+    (in_bom yes) (on_board yes)
+    (property "Reference" "P35" (id 0) (at 281.94 116.84 0))
+    (property "Value" "Pad" (id 1) (at 285.75 119.38 0)
+      (effects (font (size 1.27 1.27)) hide)
+    )
+    (property "Footprint" "hellen-one-common:PAD-TH" (id 2) (at 285.75 120.65 0)
+      (effects (font (size 1.27 1.27)) hide)
+    )
+    (property "Datasheet" "~" (id 3) (at 285.75 116.84 0)
+      (effects (font (size 1.27 1.27)) hide)
+    )
+    (pin "1")
+  )
   (symbol (lib_id "hellen-one-common:Pad") (at 285.75 124.46 0) (mirror y) (unit 1)
     (in_bom yes) (on_board yes)
@@
     (pin "1")
   )
+  (symbol (lib_id "hellen-one-common:Pad") (at 285.75 167.64 0) (mirror y) (unit 1)
+    (in_bom yes) (on_board yes)
+    (property "Reference" "P34" (id 0) (at 281.94 167.64 0))
+    (property "Value" "Pad" (id 1) (at 285.75 170.18 0)
+      (effects (font (size 1.27 1.27)) hide)
+    )
+    (property "Footprint" "hellen-one-common:PAD-TH" (id 2) (at 285.75 171.45 0)
+      (effects (font (size 1.27 1.27)) hide)
+    )
+    (property "Datasheet" "~" (id 3) (at 285.75 167.64 0)
+      (effects (font (size 1.27 1.27)) hide)
+    )
+    (pin "1")
+  )
   (symbol (lib_id "hellen-one-common:Pad") (at 285.75 172.72 0) (mirror y) (unit 1)
     (in_bom yes) (on_board yes)
@@
     (pin "1")
   )
+  (symbol (lib_id "hellen-one-common:Pad") (at 289.56 280.67 0) (mirror y) (unit 1)
+    (in_bom yes) (on_board yes)
+    (property "Reference" "P36" (id 0) (at 285.75 280.67 0))
+    (property "Value" "Pad" (id 1) (at 289.56 283.21 0)
+      (effects (font (size 1.27 1.27)) hide)
+    )
+    (property "Footprint" "hellen-one-common:PAD-TH" (id 2) (at 289.56 284.48 0)
+      (effects (font (size 1.27 1.27)) hide)
+    )
+    (property "Datasheet" "~" (id 3) (at 289.56 280.67 0)
+      (effects (font (size 1.27 1.27)) hide)
+    )
+    (pin "1")
+  )
   (symbol (lib_id "hellen-one-common:Pad") (at 290.83 300.99 180) (unit 1)
     (in_bom yes) (on_board yes)
@@
     (pin "2")
   )
+  (symbol (lib_id "hellen-one-common:Jumper-Pad-Pad") (at 110.49 95.25 0) (mirror y) (unit 1)
+    (in_bom yes) (on_board yes)
+    (property "Reference" "R8" (id 0) (at 105.7139 94.2785 0)
+      (effects (font (size 1.016 1.016)))
+    )
+    (property "Value" "Jumper-Pad-Pad" (id 1) (at 110.49 97.028 0)
+      (effects (font (size 1.016 1.016)) hide)
+    )
+    (property "Footprint" "hellen-one-common:PAD-0805-PAD" (id 2) (at 110.49 99.06 0)
+      (effects (font (size 1.524 1.524)) hide)
+    )
+    (property "Datasheet" "" (id 3) (at 110.49 95.25 0)
+      (effects (font (size 1.524 1.524)) hide)
+    )
+    (property "LCSC" " C17477" (id 4) (at 110.49 99.06 0)
+      (effects (font (size 1.27 1.27)) hide)
+    )
+    (pin "1")
+    (pin "2")
+  )
   (symbol (lib_id "hellen-one-common:Jumper-Pad-Pad") (at 110.49 105.41 0) (mirror y) (unit 1)
     (in_bom yes) (on_board yes)
@@
       (reference "P33") (unit 1) (value "Pad") (footprint "hellen-one-common:PAD-TH")
     )
+    (path "/0efe6209-6b7d-4eef-a63f-6c4134316d90"
+      (reference "P34") (unit 1) (value "Pad") (footprint "hellen-one-common:PAD-TH")
+    )
+    (path "/18f9fbef-a2d4-42f6-bf2c-4bfe788df46a"
+      (reference "P35") (unit 1) (value "Pad") (footprint "hellen-one-common:PAD-TH")
+    )
+    (path "/de670ed1-8616-46df-a756-7ba255fb3d2f"
+      (reference "P36") (unit 1) (value "Pad") (footprint "hellen-one-common:PAD-TH")
+    )
     (path "/a1ceb4d6-d412-4dc3-b899-3531d409f675"
       (reference "P38") (unit 1) (value "Pad") (footprint "hellen-one-common:PAD-TH")
@@
       (reference "R7") (unit 1) (value "20k") (footprint "hellen-one-common:R0603-4")
     )
+    (path "/f1cdedec-88f3-4b15-a07f-5ca76532bc14"
+      (reference "R8") (unit 1) (value "Jumper-Pad-Pad") (footprint "hellen-one-common:PAD-0805-PAD")
+    )
     (path "/cc637294-10be-4d8c-b760-3cd433b682b8"

Commit message: ETB-8pin + fix silkscreen
Parts:
- added P37, P39, P40, P41, P42, P45, P46: Pad, hellen-one-common:PAD-TH, symbol hellen-one-common:Pad
- J6: footprint hellen-one-common:PinHeader_1x06_P2.54mm_Vertical -> hellen-one-common:PinHeader_1x08_P2.54mm_Vertical; symbol Connector_Generic:Conn_01x06 -> Connector_Generic:Conn_01x08
Connections:
- net +5VA: now also J6.2 (Pin_2)
- net 3H: now also P2.55 (3H), P40.1 (Pin_1)
- net GNDA: now also J6.7 (Pin_7), J6.8 (Pin_8); no longer J6.6 (Pin_6)
- net IN_PPS: now also J6.5 (Pin_5); no longer J6.4 (Pin_4)
- net IN_TEMP_OR_PPS2: now also J6.6 (Pin_6); no longer J6.5 (Pin_5)
- net IN_TPS: now also J6.3 (Pin_3); no longer J6.2 (Pin_2)
- net IN_TPS2: now also J6.4 (Pin_4); no longer J6.3 (Pin_3)
- net OUT_VICS: now also P46.1 (Pin_1)
- net 2E: now reaches P2.25 (2E)
- net 2E: now also P45.1 (Pin_1)
- net 2H: now reaches P2.34 (2H)
- net 2H: now also P42.1 (Pin_1)
- net 2J: now reaches P2.35 (2J)
- net 2J: now also P41.1 (Pin_1)
- net 3M: now reaches P2.45 (3M)
- net 3M: now also P39.1 (Pin_1)
- net 3O: now reaches P2.46 (3O)
- net 3O: now also P37.1 (Pin_1)
- net 3P: now reaches P2.59 (3P), P53.1 (Pin_1)
- net 1Q renamed IN_BRAKE

Commit message: Knock jack is now DNP + fresh kicad exports
Parts:
- J25: value AudioJack3_SwitchTR -> (DNP); LCSC C165947 -> (none)
Changed lines of the file:
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@@
     (stroke (width 0) (type solid) (color 0 0 0 0))
   )
-  (wire (pts (xy 115.57 110.49) (xy 204.47 110.49))
+  (wire (pts (xy 115.57 110.49) (xy 205.74 110.49))
     (stroke (width 0) (type solid) (color 0 0 0 0))
   )
@@
     (stroke (width 0) (type solid) (color 0 0 0 0))
   )
-  (wire (pts (xy 132.08 151.13) (xy 203.2 151.13))
+  (wire (pts (xy 132.08 151.13) (xy 248.92 151.13))
     (stroke (width 0) (type solid) (color 0 0 0 0))
   )
@@
     (stroke (width 0) (type solid) (color 0 0 0 0))
   )
-  (wire (pts (xy 196.85 107.95) (xy 255.27 107.95))
-    (stroke (width 0) (type solid) (color 0 0 0 0))
-  )
   (wire (pts (xy 196.85 196.85) (xy 132.08 196.85))
     (stroke (width 0) (type solid) (color 0 0 0 0))
@@
     (stroke (width 0) (type solid) (color 0 0 0 0))
   )
+  (wire (pts (xy 205.74 97.79) (xy 205.74 100.33))
+    (stroke (width 0) (type solid) (color 0 0 0 0))
+  )
+  (wire (pts (xy 205.74 100.33) (xy 245.11 100.33))
+    (stroke (width 0) (type solid) (color 0 0 0 0))
+  )
+  (wire (pts (xy 205.74 101.6) (xy 205.74 110.49))
+    (stroke (width 0) (type solid) (color 0 0 0 0))
+  )
   (wire (pts (xy 205.74 186.69) (xy 132.08 186.69))
     (stroke (width 0) (type solid) (color 0 0 0 0))
@@
     (stroke (width 0) (type solid) (color 0 0 0 0))
   )
+  (wire (pts (xy 245.11 100.33) (xy 245.11 107.95))
+    (stroke (width 0) (type solid) (color 0 0 0 0))
+  )
+  (wire (pts (xy 245.11 107.95) (xy 255.27 107.95))
+    (stroke (width 0) (type solid) (color 0 0 0 0))
+  )
   (wire (pts (xy 245.11 111.76) (xy 309.88 111.76))
     (stroke (width 0) (type solid) (color 0 0 0 0))
@@
     (stroke (width 0) (type solid) (color 0 0 0 0))
   )
+  (wire (pts (xy 248.92 160.02) (xy 248.92 151.13))
+    (stroke (width 0) (type solid) (color 0 0 0 0))
+  )
   (wire (pts (xy 248.92 160.02) (xy 309.88 160.02))
     (stroke (width 0) (type solid) (color 0 0 0 0))
@@
     (stroke (width 0) (type solid) (color 0 0 0 0))
   )
+  (wire (pts (xy 271.78 101.6) (xy 205.74 101.6))
+    (stroke (width 0) (type solid) (color 0 0 0 0))
+  )
+  (wire (pts (xy 271.78 119.38) (xy 271.78 101.6))
+    (stroke (width 0) (type solid) (color 0 0 0 0))
+  )
   (wire (pts (xy 271.78 119.38) (xy 309.88 119.38))
     (stroke (width 0) (type solid) (color 0 0 0 0))
@@
     (effects (font (size 1.27 1.27)) (justify left bottom))
   )
+  (text "Not OEM" (at 133.35 156.21 0)
+    (effects (font (size 1.27 1.27)) (justify left bottom))
+  )
   (text "Not OEM" (at 133.35 179.07 0)
     (effects (font (size 1.27 1.27)) (justify left bottom))
@@
       (effects (font (size 1.27 1.27)) (justify right))
     )
-    (property "Value" "AudioJack3_SwitchTR" (id 1) (at 243.3321 328.5628 0)
+    (property "Value" "(DNP)" (id 1) (at 243.3321 328.5628 0)
       (effects (font (size 1.27 1.27)) (justify right))
     )
@@
       (effects (font (size 1.27 1.27)) hide)
     )
-    (property "LCSC" "C165947" (id 4) (at 246.38 322.58 0)
+    (property "LCSC" "" (id 4) (at 246.38 322.58 0)
       (effects (font (size 1.27 1.27)) hide)
     )
@@
     )
     (path "/42701a5c-235d-4e1c-b394-77856f0b91bb"
-      (reference "J25") (unit 1) (value "AudioJack3_SwitchTR") (footprint "hellen-one-common:Jack_3.5mm_PJ-3250-5A")
+      (reference "J25") (unit 1) (value "(DNP)") (footprint "hellen-one-common:Jack_3.5mm_PJ-3250-5A")
     )
     (path "/ab5a9649-4542-4cc5-95df-391b2db17a5e"
